File: board/Electronicsmb.brd (EAGLE design)
At the start: 96 x 70 mm, 37 parts

Commit message: larger drill holes and points for positive and negative
Parts:
- added J2, J3: (no value), SparkFun-Connectors:1X02
- moved R3 2.54 mm to (44.5, 58.4)
Connections:
- net GND: now also J3.1, J3.2
- net VCC: now also J2.1, J2.2
Routing:
- net VCC: track 108.9 -> 117.9 mm
- net GND: track 269.9 -> 278.9 mm
- net D11: track 13.6 -> 11.6 mm
- net N$25: track 13.3 -> 14.4 mm
Other:
- board text added: "+"
- board text added: "-"
- board text added: "BRAVE"
- board text added: "Battery"
- board text added: "CHEERFUL"
- board text added: "CLEAN"
- board text added: "COURTEOUS"
- board text added: "FRIENDLY"
- board text added: "HELPFUL"
- board text added: "KIND"
- board text added: "LOYAL"
- board text added: "OBEDIENT"
- board text added: "REVERENT"
- board text added: "THRIFTY"
- board text added: "TRUSTWORTHY"
Changed lines of the file:
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@@
 <text x="86.36" y="2.54" size="1.778" layer="25">Mode</text>
 <text x="2.54" y="10.16" size="1.778" layer="25">Pin 13 LED</text>
-<hole x="6.35" y="6.35" drill="1.5"/>
-<hole x="6.35" y="64.77" drill="1.5"/>
-<hole x="88.9" y="64.77" drill="1.5"/>
-<hole x="88.9" y="6.35" drill="1.5"/>
+<hole x="6.35" y="6.35" drill="3"/>
+<hole x="6.35" y="64.77" drill="3"/>
+<hole x="88.9" y="64.77" drill="3"/>
+<hole x="88.9" y="6.35" drill="3"/>
+<text x="58.42" y="66.04" size="1.778" layer="25">TRUSTWORTHY</text>
+<text x="72.39" y="52.07" size="1.778" layer="25">LOYAL</text>
+<text x="73.66" y="39.37" size="1.778" layer="25">HELPFUL</text>
+<text x="71.12" y="26.67" size="1.778" layer="25">FRIENDLY</text>
+<text x="59.69" y="15.24" size="1.778" layer="25">COURTEOUS</text>
+<text x="44.45" y="10.16" size="1.778" layer="25">KIND</text>
+<text x="25.4" y="5.08" size="1.778" layer="25">OBEDIENT</text>
+<text x="12.7" y="26.67" size="1.778" layer="25">CHEERFUL</text>
+<text x="10.16" y="39.37" size="1.778" layer="25">THRIFTY</text>
+<text x="15.24" y="52.07" size="1.778" layer="25">BRAVE</text>
+<text x="25.4" y="66.04" size="1.778" layer="21">CLEAN</text>
+<text x="40.64" y="60.96" size="1.778" layer="25">REVERENT</text>
+<text x="8.89" y="67.31" size="1.778" layer="21">Battery</text>
+<text x="5.08" y="55.88" size="2.54" layer="21">+</text>
+<text x="16.51" y="55.88" size="2.54" layer="21">-</text>
 </plain>
 <attributes>
@@
 <element name="R14" library="resistor" library_urn="urn:adsk.eagle:library:348" package="0204/7" package3d_urn="urn:adsk.eagle:package:25945/1" value="270" x="64.77" y="19.05"/>
 <element name="R2" library="resistor" library_urn="urn:adsk.eagle:library:348" package="0204/7" package3d_urn="urn:adsk.eagle:package:25945/1" value="270" x="29.21" y="55.88" rot="R180"/>
-<element name="R3" library="resistor" library_urn="urn:adsk.eagle:library:348" package="0204/7" package3d_urn="urn:adsk.eagle:package:25945/1" value="270" x="44.45" y="60.96" rot="R180"/>
+<element name="R3" library="resistor" library_urn="urn:adsk.eagle:library:348" package="0204/7" package3d_urn="urn:adsk.eagle:package:25945/1" value="270" x="44.45" y="58.42" rot="R180"/>
 <element name="R4" library="resistor" library_urn="urn:adsk.eagle:library:348" package="0204/7" package3d_urn="urn:adsk.eagle:package:25945/1" value="270" x="64.77" y="53.34"/>
 <element name="R6" library="resistor" library_urn="urn:adsk.eagle:library:348" package="0204/7" package3d_urn="urn:adsk.eagle:package:25945/1" value="270" x="64.77" y="49.53"/>
@@
 <element name="U$1" library="Arduino-clone" package="NANO" value="NANO" x="48.26" y="25.4"/>
 <element name="U$2" library="homemadehamcustom" package="TT_POT" value="TT_POT_P090L" x="73.66" y="10.16" rot="R270"/>
+<element name="J2" library="SparkFun-Connectors" library_urn="urn:adsk.eagle:library:513" package="1X02" package3d_urn="urn:adsk.eagle:package:38039/1" value="" x="8.89" y="55.88" rot="R90"/>
+<element name="J3" library="SparkFun-Connectors" library_urn="urn:adsk.eagle:library:513" package="1X02" package3d_urn="urn:adsk.eagle:package:38039/1" value="" x="13.97" y="55.88" rot="R90"/>
 </elements>
 <signals>
@@
 <wire x1="67.2084" y1="61.2648" x2="67.31" y2="61.25" width="0.1524" layer="1"/>
 <wire x1="48.3108" y1="65.9892" x2="48.27" y2="66" width="0.1524" layer="1"/>
+<contactref element="J3" pad="2"/>
+<contactref element="J3" pad="1"/>
+<wire x1="14.0208" y1="58.3692" x2="14.0208" y2="55.9308" width="0.1524" layer="1"/>
+<wire x1="14.0208" y1="55.9308" x2="13.97" y2="55.88" width="0.1524" layer="1"/>
+<wire x1="14.0208" y1="58.3692" x2="13.97" y2="58.42" width="0.1524" layer="1"/>
+<wire x1="14.0208" y1="64.77" x2="14.0208" y2="58.5216" width="0.1524" layer="1"/>
+<wire x1="14.0208" y1="58.5216" x2="13.97" y2="58.42" width="0.1524" layer="1"/>
+<wire x1="14.0208" y1="64.77" x2="13.97" y2="64.77" width="0.1524" layer="1"/>
 </signal>
 <signal name="VCC">
@@
 <wire x1="19.3548" y1="47.0916" x2="30.7848" y2="35.6616" width="0.1524" layer="16"/>
 <wire x1="19.3548" y1="56.8452" x2="19.3548" y2="47.0916" width="0.1524" layer="16"/>
-<wire x1="11.43" y1="64.77" x2="19.3548" y2="56.8452" width="0.1524" layer="16"/>
+<wire x1="11.43" y1="64.77" x2="13.2588" y2="62.9412" width="0.1524" layer="16"/>
+<wire x1="13.2588" y1="62.9412" x2="19.3548" y2="56.8452" width="0.1524" layer="16"/>
 <wire x1="38.1" y1="24.2316" x2="38.1" y2="24.13" width="0.1524" layer="16"/>
 <wire x1="76.5048" y1="4.572" x2="76.2" y2="4.572" width="0.1524" layer="16"/>
@@
 <wire x1="76.2" y1="4.572" x2="76.16" y2="4.46" width="0.1524" layer="16"/>
 <wire x1="38.1" y1="24.0792" x2="38.1" y2="24.13" width="0.1524" layer="16"/>
+<contactref element="J2" pad="2"/>
+<contactref element="J2" pad="1"/>
+<wire x1="8.9916" y1="58.3692" x2="8.9916" y2="55.9308" width="0.1524" layer="1"/>
+<wire x1="8.9916" y1="55.9308" x2="8.89" y2="55.88" width="0.1524" layer="1"/>
+<wire x1="8.9916" y1="58.3692" x2="8.89" y2="58.42" width="0.1524" layer="1"/>
+<wire x1="13.2588" y1="62.7888" x2="8.9916" y2="58.5216" width="0.1524" layer="16"/>
+<wire x1="13.2588" y1="62.9412" x2="13.2588" y2="62.7888" width="0.1524" layer="16"/>
+<wire x1="8.9916" y1="58.5216" x2="8.89" y2="58.42" width="0.1524" layer="16"/>
 </signal>
 <signal name="N$15">
@@
 <contactref element="R3" pad="2"/>
 <contactref element="D11" pad="A"/>
-<wire x1="32.1564" y1="60.96" x2="40.5384" y2="60.96" width="0.1524" layer="1"/>
 <wire x1="31.242" y1="60.0456" x2="32.1564" y2="60.96" width="0.1524" layer="1"/>
 <wire x1="29.4132" y1="60.0456" x2="31.242" y2="60.0456" width="0.1524" layer="1"/>
 <wire x1="28.3464" y1="61.1124" x2="29.4132" y2="60.0456" width="0.1524" layer="1"/>
-<wire x1="40.5384" y1="60.96" x2="40.64" y2="60.96" width="0.1524" layer="1"/>
 <wire x1="28.3464" y1="61.1124" x2="28.21" y2="61.25" width="0.1524" layer="1"/>
+<wire x1="34.5948" y1="58.5216" x2="40.5384" y2="58.5216" width="0.1524" layer="1"/>
+<wire x1="32.1564" y1="60.96" x2="34.5948" y2="58.5216" width="0.1524" layer="1"/>
+<wire x1="40.5384" y1="58.5216" x2="40.64" y2="58.42" width="0.1524" layer="1"/>
 </signal>
 <signal name="N$26">
@@
 <wire x1="53.34" y1="50.1396" x2="53.34" y2="49.53" width="0.1524" layer="1"/>
 <wire x1="48.3108" y1="55.1688" x2="53.34" y2="50.1396" width="0.1524" layer="1"/>
-<wire x1="48.3108" y1="60.96" x2="48.3108" y2="55.1688" width="0.1524" layer="1"/>
-<wire x1="48.3108" y1="60.96" x2="48.26" y2="60.96" width="0.1524" layer="1"/>
+<wire x1="48.3108" y1="58.3692" x2="48.3108" y2="55.1688" width="0.1524" layer="1"/>
+<wire x1="53.34" y1="50.1396" x2="53.34" y2="49.53" width="0.1524" layer="1"/>
+<wire x1="48.3108" y1="58.3692" x2="48.26" y2="58.42" width="0.1524" layer="1"/>
 </signal>
 <signal name="D10">

Commit message: minor tweaks
Connections:
- new net RAW: J1.2, U$1.RAW
- net VCC: no longer J1.2
Routing:
- net RAW: track 0.00 -> 59.3 mm
- net GND: track 278.9 -> 272.4 mm
- net VCC: track 117.9 -> 121.9 mm
- net N$23: track 62.1 -> 61.1 mm
- net N$25: track 14.4 -> 13.6 mm
- net D11: track 11.6 -> 11.0 mm

Commit message: final tweaks to V1 and starter code
Parts:
- removed A1, A2, A3: (no value), wirepad:2,54/1,0
- added J4: (no value), SparkFun-Connectors:1X04
- R1, R10, R11, R12, R13, R14, R2, R3, R4, R6, R7, R8, R9: device resistor:0204/7 -> SparkFun:AXIAL-0.4
- moved A4 10.2 mm to (29.2, 44.5)
- moved A5 8.89 mm to (29.2, 38.1)
- moved A6 7.62 mm to (29.2, 31.8)
- moved A7 7.62 mm to (29.2, 25.4)
- renumbered D1 to D15, D13 to D16
Connections:
- removed net D1: R14.1, U$1.RX1
- removed net N$1: S1.2, U$1.TX0
- new net RX: J4.2, U$1.RX1
- new net TX: J4.3, U$1.TX0
- net A1: now also R14.P$1; no longer A1.1
- net A2: now also R2.P$1; no longer A2.1
- net A3: now also S1.2; no longer A3.1
- net D10: now also R4.P$1; no longer R4.1
- net D11: now also R3.P$1; no longer R3.1
- net D12: now also R1.P$1; no longer R1.1
- net D13: no longer R2.1
- net D2: now also R13.P$1; no longer R13.1
- net D3: now also R12.P$1; no longer R12.1
- net D4: now also R11.P$1; no longer R11.1
- net D5: now also R10.P$1; no longer R10.1
- net D6: now also R9.P$1; no longer R9.1
- net D7: now also R8.P$1; no longer R8.1
- net D8: now also R7.P$1; no longer R7.1
- net D9: now also R6.P$1; no longer R6.1
- net GND: now also J4.1
- net N$13: now also R2.P$2; no longer R2.2
- net N$15: now also R14.P$2; no longer R14.2
- net N$16: now also R13.P$2; no longer R13.2
- net N$17: now also R12.P$2; no longer R12.2
- net N$18: now also R11.P$2; no longer R11.2
- net N$19: now also R10.P$2; no longer R10.2
- net N$20: now also R9.P$2; no longer R9.2
- net N$21: now also R8.P$2; no longer R8.2
- net N$22: now also R7.P$2; no longer R7.2
- net N$23: now also R6.P$2; no longer R6.2
- net N$24: now also R4.P$2; no longer R4.2
- net N$25: now also R3.P$2; no longer R3.2
- net N$26: now also R1.P$2; no longer R1.2
- net VCC: now also J4.4
Routing:
- net N$1: track 37.4 -> 0.00 mm
- net A3: track 9.97 -> 40.1 mm
- net A1: track 12.0 -> 33.7 mm
- net VCC: track 121.9 -> 103.1 mm
- net RX: track 0.00 -> 18.2 mm
- net TX: track 0.00 -> 14.6 mm
- net N$20: track 44.1 -> 56.5 mm
- net GND: track 272.4 -> 283.8 mm
- net N$24: track 54.9 -> 64.8 mm
- net RAW: track 59.3 -> 67.4 mm
- net D1: track 7.62 -> 0.00 mm
- net A2: track 11.1 -> 18.1 mm
- net D13: track 6.71 -> 0.00 mm
- net N$23: track 61.1 -> 67.5 mm
- net A4: track 8.89 -> 13.8 mm
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Other:
- board text added: "Pin 16 LED"
- board text removed: "Pin 13 LED"
